File: hardware/efm32hg309_board.kicad_pcb (KiCad board)
At the start: 2 copper layers, 17.8 x 22.9 mm, 12 parts, among them J1 USB_OTG, P1 CONN_01X09, P2 CONN_01X09, SW1 RST, U1 EFM32HG309

Commit message: cleaned up board
Routing:
- net +5V: track 18.4 -> 19.2 mm
Changed lines of the file:
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@@
     (links 49)
     (no_connects 0)
-    (area 138.379999 96.469999 156.260001 119.430001)
+    (area 134.686667 93.569 159.953334 122.795)
     (thickness 1.6)
     (drawings 24)
-    (tracks 157)
+    (tracks 158)
     (zones 0)
     (modules 12)
@@
     (tags "QFN 0.65")
     (attr smd)
-    (fp_text reference U1 (at 0 -3.7 90) (layer F.SilkS)
+    (fp_text reference U1 (at -9.525 0 180) (layer F.SilkS)
       (effects (font (size 1 1) (thickness 0.15)))
     )
@@
     )
   )
+  (gr_text EFM32HG309 (at 147.32 116.078) (layer F.SilkS)
+    (effects (font (size 0.5 0.5) (thickness 0.1)))
+  )
   (gr_text GND (at 141.732 97.79) (layer F.SilkS)
     (effects (font (size 0.5 0.5) (thickness 0.1)))
@@
     (effects (font (size 0.5 0.5) (thickness 0.1)))
   )
-  (gr_text "EFM32HG309 BOARD v0.3\nBy: Jonas 'Kokjo' Rudloff\nEmail: jonas.t.rudloff@gmail.com\n" (at 151.765 107.95 270) (layer B.SilkS)
+  (gr_text "EFM32HG309 BOARD v0.3\nBy: Jonas 'Kokjo' Rudloff\nEmail: jonas.t.rudloff@gmail.com" (at 151.765 107.95 270) (layer B.SilkS)
     (effects (font (size 0.7 0.7) (thickness 0.1)) (justify mirror))
-  )
-  (gr_text EFM32HG309 (at 147.32 121.92) (layer F.SilkS)
-    (effects (font (size 1 1) (thickness 0.15)))
   )
   (gr_line (start 156.21 96.52) (end 138.43 96.52) (layer Edge.Cuts) (width 0.1))
@@
   (via (at 148.945 110.07) (size 0.6) (drill 0.4) (layers F.Cu B.Cu) (net 2))
   (via (at 146.995 110.07) (size 0.6) (drill 0.4) (layers F.Cu B.Cu) (net 2))
-  (segment (start 147.645 109.213243) (end 147.645 110.07) (width 0.25) (layer F.Cu) (net 3))
-  (segment (start 149.1 105.14) (end 147.645 106.595) (width 0.25) (layer F.Cu) (net 3))
-  (segment (start 147.645 106.595) (end 147.645 109.213243) (width 0.25) (layer F.Cu) (net 3))
-  (segment (start 149.225 105.14) (end 149.1 105.14) (width 0.25) (layer F.Cu) (net 3))
+  (segment (start 148.274999 106.004449) (end 148.284926 106.004449) (width 0.25) (layer F.Cu) (net 3))
+  (segment (start 149.149375 105.14) (end 149.225 105.14) (width 0.25) (layer F.Cu) (net 3))
+  (segment (start 148.284926 106.004449) (end 149.149375 105.14) (width 0.25) (layer F.Cu) (net 3))
+  (segment (start 148.62 102.034998) (end 148.274999 102.379999) (width 0.25) (layer F.Cu) (net 3))
+  (segment (start 148.274999 102.379999) (end 148.274999 106.004449) (width 0.25) (layer F.Cu) (net 3))
+  (segment (start 148.274999 106.004449) (end 147.645 106.634448) (width 0.25) (layer F.Cu) (net 3))
+  (segment (start 147.645 106.634448) (end 147.645 108.815001) (width 0.25) (layer F.Cu) (net 3))
+  (segment (start 147.645 108.815001) (end 147.645 110.07) (width 0.25) (layer F.Cu) (net 3))
+  (segment (start 154.94 100.33) (end 153.674 100.33) (width 0.25) (layer F.Cu) (net 3))
+  (segment (start 153.674 100.33) (end 151.969002 102.034998) (width 0.25) (layer F.Cu) (net 3))
+  (segment (start 151.969002 102.034998) (end 148.62 102.034998) (width 0.25) (layer F.Cu) (net 3))
   (segment (start 148.62 100.704) (end 148.62 102.034998) (width 0.25) (layer F.Cu) (net 3))
-  (segment (start 148.62 102.034998) (end 148.274999 102.379999) (width 0.25) (layer F.Cu) (net 3))
-  (segment (start 148.274999 102.379999) (end 148.274999 104.314999) (width 0.25) (layer F.Cu) (net 3))
-  (segment (start 148.274999 104.314999) (end 149.1 105.14) (width 0.25) (layer F.Cu) (net 3))
   (segment (start 148.62 100.704) (end 148.62 101.644) (width 0.25) (layer F.Cu) (net 3))
-  (segment (start 153.398599 101.719001) (end 154.7876 100.33) (width 0.25) (layer F.Cu) (net 3))
-  (segment (start 148.62 101.644) (end 148.695001 101.719001) (width 0.25) (layer F.Cu) (net 3))
-  (segment (start 148.695001 101.719001) (end 153.398599 101.719001) (width 0.25) (layer F.Cu) (net 3))
   (segment (start 154.7876 100.33) (end 154.94 100.33) (width 0.25) (layer F.Cu) (net 3))
   (segment (start 145.695 110.07) (end 145.695 109.845) (width 0.25) (layer F.Cu) (net 4))
