File: hardware/efm32hg309_board.sch (KiCad schematic (older format))
At the start: 12 parts, among them J1 USB_OTG, P1 CONN_01X09, P2 CONN_01X09, SW1 RST, U1 EFM32HG309

Commit message: cleaned up board
Connections:
- net GND: no longer J1.6 (Shield)
Changed lines of the file:
@@
 $EndComp
 $Comp
-L +3V3 #PWR3
+L +3V3 #PWR01
 U 1 1 5A79BEC6
 P 7100 3800
-F 0 "#PWR3" H 7100 3650 50  0001 C CNN
+F 0 "#PWR01" H 7100 3650 50  0001 C CNN
 F 1 "+3V3" H 7100 3940 50  0000 C CNN
 F 2 "" H 7100 3800 50  0000 C CNN
@@
 $EndComp
 $Comp
-L +5V #PWR4
+L +5V #PWR02
 U 1 1 5A79C1DB
 P 7875 3050
-F 0 "#PWR4" H 7875 2900 50  0001 C CNN
+F 0 "#PWR02" H 7875 2900 50  0001 C CNN
 F 1 "+5V" H 7875 3190 50  0000 C CNN
 F 2 "" H 7875 3050 50  0000 C CNN
@@
 Connection ~ 7875 3150
 $Comp
-L GND #PWR5
+L GND #PWR03
 U 1 1 5AD23389
 P 7875 4475
-F 0 "#PWR5" H 7875 4225 50  0001 C CNN
+F 0 "#PWR03" H 7875 4225 50  0001 C CNN
 F 1 "GND" H 7875 4325 50  0000 C CNN
 F 2 "" H 7875 4475 50  0001 C CNN
@@
 $EndComp
 $Comp
-L GND #PWR1
+L GND #PWR04
 U 1 1 5ADC77D0
 P 5425 4725
-F 0 "#PWR1" H 5425 4475 50  0001 C CNN
+F 0 "#PWR04" H 5425 4475 50  0001 C CNN
 F 1 "GND" H 5425 4575 50  0000 C CNN
 F 2 "" H 5425 4725 50  0001 C CNN
@@
 $EndComp
 $Comp
-L GND #PWR2
+L GND #PWR05
 U 1 1 5ADCD8D9
 P 5475 5500
-F 0 "#PWR2" H 5475 5250 50  0001 C CNN
+F 0 "#PWR05" H 5475 5250 50  0001 C CNN
 F 1 "GND" H 5475 5350 50  0000 C CNN
 F 2 "" H 5475 5500 50  0001 C CNN
@@
 Wire Wire Line
 	7250 3700 7250 4400
+Connection ~ 7250 3975
+Wire Wire Line
+	6925 3375 7250 3600
+Wire Wire Line
+	6925 3500 7250 3500
+Wire Wire Line
+	7550 3975 7250 3975
 Wire Wire Line
 	7550 3900 7550 3975
-Wire Wire Line
-	7250 3975 7650 3975
-Connection ~ 7250 3975
-Wire Wire Line
-	7650 3975 7650 3900
-Connection ~ 7550 3975
-Wire Wire Line
-	6925 3375 7250 3600
-Wire Wire Line
-	6925 3500 7250 3500
 $EndSCHEMATC
